File: PCB/keyboard.kicad_sch (KiCad schematic)
At the start: 217 parts, among them J1 USB_C_Receptacle, SW1 1, SW10 30, SW11 44, SW12 69, SW13 26, SW14 25, SW15 3, SW16 17, SW17 31, SW18 45, SW19 59, SW2 15, SW20 40, SW21 39, SW22 4, SW23 18, SW24 32, SW25 46, SW27 54, SW28 53, SW29 5, SW3 29, SW30 19, SW31 33, SW32 47, SW33 61, SW34 68, SW36 6, SW37 20, SW38 34, SW39 48, SW4 43, SW41 13, SW42 27, SW43 7, SW44 21, SW45 35, SW48 41, SW49 SW_SPDT, SW5 57, SW50 8, SW51 22, SW52 36, SW55 55, SW57 9, SW58 23, SW59 37, SW6 12, SW60 51, SW61 65, SW62 14, SW63 28, SW64 10, SW65 24, SW66 38, SW67 52, SW68 66, SW7 11, SW70 56, SW71 70, SW8 2, SW9 16, U1 TP4056-42-ESOP8, U3 MCP1700x-330xxTO

Commit message: LED
Parts:
- D100, D101, D102, D104, D105, D106, D107, D108, D109, D110, D111, D112, D113, D114, D115, D116, D117, D118, D119, D12, D120, D121, D122, D123, D124, D125, D126, D127, D128, D129, D130, D131, D132, D134, D137, D138, D139, D26, D35, D40, D46, D47, D49, D53, D54, D56, D62, D63, D70, D71, D72, D73, D74, D75, D76, D77, D78, D79, D80, D81, D82, D83, D84, D85, D86, D87, D88, D89, D90, D91, D92, D93, D94, D95, D96, D97, D98, D99: footprint LED_SMD:LED_SK6812MINI_PLCC4_3.5x3.5mm_P1.75mm -> led:SK6812MINI-E_fixed

Commit message: hiojb
Parts:
- SW49: footprint Button_Switch_THT:SW_CK_JS202011CQN_DPDT_Straight -> sw slide:SW_Slide_1P2T_CK_OS102011MS2Q
Changed lines of the file:
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@@
 			)
 		)
-		(property "Footprint" "Button_Switch_THT:SW_CK_JS202011CQN_DPDT_Straight"
+		(property "Footprint" "sw slide:SW_Slide_1P2T_CK_OS102011MS2Q"
 			(at 220.98 38.1 0)
 			(effects
