File: PCB/keyboard.kicad_pcb (KiCad board)
At the start: 2 copper layers, 314.8 x 99 mm, 217 parts, among them J1 USB_C_Receptacle, SW1 1, SW10 30, SW11 44, SW12 69, SW13 26, SW14 25, SW15 3, SW16 17, SW17 31, SW18 45, SW19 59, SW2 15, SW20 40, SW21 39, SW22 4, SW23 18, SW24 32, SW25 46, SW27 54, SW28 53, SW29 5, SW3 29, SW30 19, SW31 33, SW32 47, SW33 61, SW34 68, SW36 6, SW37 20, SW38 34, SW39 48, SW4 43, SW41 13, SW42 27, SW43 7, SW44 21, SW45 35, SW48 41, SW49 SW_SPDT, SW5 57, SW50 8, SW51 22, SW52 36, SW55 55, SW57 9, SW58 23, SW59 37, SW6 12, SW60 51, SW61 65, SW62 14, SW63 28, SW64 10, SW65 24, SW66 38, SW67 52, SW68 66, SW7 11, SW70 56, SW71 70, SW8 2, SW9 16, U1 TP4056-42-ESOP8, U3 MCP1700x-330xxTO

Commit message: LED
Parts:
- D100, D101, D102, D104, D105, D106, D107, D108, D109, D110, D111, D112, D113, D114, D115, D116, D117, D118, D119, D12, D120, D121, D122, D123, D124, D125, D126, D127, D128, D129, D130, D131, D132, D134, D137, D138, D139, D26, D35, D40, D46, D47, D49, D53, D54, D56, D62, D63, D70, D71, D72, D73, D74, D75, D76, D77, D78, D79, D80, D81, D82, D83, D84, D85, D86, D87, D88, D89, D90, D91, D92, D93, D94, D95, D96, D97, D98, D99: footprint LED_SMD:LED_SK6812MINI_PLCC4_3.5x3.5mm_P1.75mm -> led:SK6812MINI-E_fixed
- moved D113 11.5 mm to (273.6, 31.3)
- moved D71 6.08 mm to (294.0, 18.7)
- moved D120 4.53 mm to (131.0, 89.3)
- moved D118 4.41 mm to (169.4, 89.1)
- moved D117 3.12 mm to (187.1, 88.6)
- moved D119 2.57 mm to (148.8, 88.4)
- moved D130 2.06 mm to (160.5, 69.4)
- moved D26 1.86 mm to (86.9, 89.0)
- moved D125 1.73 mm to (293.6, 87.3)
- moved D72 1.48 mm to (261.2, 12.3)
- moved D124 1.47 mm to (293.7, 71.8)
- moved D40 1.43 mm to (52.1, 88.4)
- moved D104 1.24 mm to (258.5, 50.5)
- moved D138 1.12 mm to (273.7, 105.1)
- moved D114 1.06 mm to (295.7, 34.1)
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Routing:
- net GND: track 1907.2 -> 1972.8 mm, vias 17 -> 40
- net col13: track 221.9 -> 176.2 mm, vias 8 -> 6
- net col1: track 433.7 -> 413.0 mm, vias 4 -> 5
- net Net-(D136-A): track 47.1 -> 67.3 mm, vias 2 -> 1
- net Net-(D112-DOUT): track 20.2 -> 36.7 mm, vias 0 -> 2
- net Net-(D33-A): track 22.4 -> 8.51 mm, vias 1 -> 0
- net Net-(D134-DOUT): track 28.1 -> 41.2 mm, vias 0 -> 4
- net Net-(D137-DOUT): track 49.0 -> 61.5 mm, vias 0 -> 4
- net Net-(D134-DIN): track 127.3 -> 139.7 mm, vias 0 -> 4
- net Net-(D138-DOUT): track 29.1 -> 41.3 mm, vias 0 -> 4
- net Net-(D54-DOUT): track 26.9 -> 38.9 mm, vias 0 -> 4
- net <NO NET>: track 1806.9 -> 1818.0 mm, vias 10 -> 80
- net Net-(D53-DOUT): track 28.4 -> 38.6 mm, vias 0 -> 4
- net col3: track 381.8 -> 390.7 mm, vias 4 -> 5
- net Net-(D123-DOUT): track 46.1 -> 54.7 mm, vias 0 -> 2
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
Commit message: update
Parts:
- added G***: LOGO, footprint:gengar3, F.Cu at (185.1, 57.4)
- added G***: LOGO, footprint:gengar2, F.Cu at (112.9, 35.9)
- added G***: LOGO, footprint:12, F.Cu at (52.7, 76.0)
- added G***: LOGO, footprint:gengar, F.Cu at (256.6, 58.0)
Other:
- board text removed: "^ Suggested board edge for RF ^"
