File: Reciever/Reciever.kicad_pcb (KiCad board)
At the start: 2 copper layers, 17.3 x 23 mm, 3 parts, among them J2 USB_A, U1 ESP32-S3-MINI-1, U2 MCP1700x-330xxTT

Commit message: UPDATING RECIEVER
Connections:
- J2 pad 2: unconnected-(J2-D--Pad2) -> D-
- J2 pad 3: unconnected-(J2-D+-Pad3) -> D+
- U1 pad 23: unconnected-(U1-USB_D--Pad23) -> D-
- U1 pad 24: unconnected-(U1-USB_D+-Pad24) -> D+
Routing:
- net D-: track 0.00 -> 4.26 mm
- net D+: track 0.00 -> 3.81 mm
Changed lines of the file:
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@@
 	(net 24 "unconnected-(U1-IO13-Pad17)")
 	(net 25 "unconnected-(U1-IO14-Pad18)")
-	(net 26 "unconnected-(U1-USB_D+-Pad24)")
+	(net 26 "D+")
 	(net 27 "unconnected-(U1-IO47-Pad27)")
 	(net 28 "unconnected-(U1-TXD0-Pad39)")
 	(net 29 "unconnected-(U1-IO18-Pad22)")
-	(net 30 "unconnected-(U1-USB_D--Pad23)")
+	(net 30 "D-")
 	(net 31 "unconnected-(U1-IO46-Pad44)")
 	(net 32 "unconnected-(U1-IO17-Pad21)")
@@
 	(net 40 "unconnected-(U1-IO2-Pad6)")
 	(net 41 "unconnected-(U1-IO12-Pad16)")
-	(net 42 "unconnected-(J2-D--Pad2)")
-	(net 43 "unconnected-(J2-D+-Pad3)")
-	(net 44 "unconnected-(J2-Shield-Pad5)")
-	(net 45 "Net-(U1-3V3)")
-	(net 46 "unconnected-(U1-IO1-Pad5)")
+	(net 42 "unconnected-(J2-Shield-Pad5)")
+	(net 43 "Net-(U1-3V3)")
+	(net 44 "unconnected-(U1-IO1-Pad5)")
 	(footprint "Connector_USB:USB_A_Molex_67643_Horizontal"
 		(layer "F.Cu")
@@
 			(layers "*.Cu" "*.Mask")
 			(remove_unused_layers no)
-			(net 42 "unconnected-(J2-D--Pad2)")
+			(net 30 "D-")
 			(pinfunction "D-")
 			(pintype "bidirectional")
@@
 			(layers "*.Cu" "*.Mask")
 			(remove_unused_layers no)
-			(net 43 "unconnected-(J2-D+-Pad3)")
+			(net 26 "D+")
 			(pinfunction "D+")
 			(pintype "bidirectional")
@@
 			(layers "*.Cu" "*.Mask")
 			(remove_unused_layers no)
-			(net 44 "unconnected-(J2-Shield-Pad5)")
+			(net 42 "unconnected-(J2-Shield-Pad5)")
 			(pinfunction "Shield")
 			(pintype "passive")
@@
 			(layers "*.Cu" "*.Mask")
 			(remove_unused_layers no)
-			(net 44 "unconnected-(J2-Shield-Pad5)")
+			(net 42 "unconnected-(J2-Shield-Pad5)")
 			(pinfunction "Shield")
 			(pintype "passive")
@@
 			(size 0.8 0.4)
 			(layers "F.Cu" "F.Mask" "F.Paste")
-			(net 45 "Net-(U1-3V3)")
+			(net 43 "Net-(U1-3V3)")
 			(pinfunction "3V3")
 			(pintype "power_in")
@@
 			(size 0.8 0.4)
 			(layers "F.Cu" "F.Mask" "F.Paste")
-			(net 46 "unconnected-(U1-IO1-Pad5)")
+			(net 44 "unconnected-(U1-IO1-Pad5)")
 			(pinfunction "IO1")
 			(pintype "bidirectional")
@@
 			(size 0.8 0.4)
 			(layers "F.Cu" "F.Mask" "F.Paste")
-			(net 30 "unconnected-(U1-USB_D--Pad23)")
+			(net 30 "D-")
 			(pinfunction "USB_D-")
 			(pintype "bidirectional")
@@
 			(size 0.8 0.4)
 			(layers "F.Cu" "F.Mask" "F.Paste")
-			(net 26 "unconnected-(U1-USB_D+-Pad24)")
+			(net 26 "D+")
 			(pinfunction "USB_D+")
 			(pintype "bidirectional")
@@
 			(layers "B.Cu" "B.Mask" "B.Paste")
 			(roundrect_rratio 0.25)
-			(net 45 "Net-(U1-3V3)")
+			(net 43 "Net-(U1-3V3)")
 			(pinfunction "VO")
 			(pintype "power_out")
@@
 	)
 	(segment
+		(start 132.74 70.61)
+		(end 132.74 66.84)
+		(width 0.2)
+		(layer "F.Cu")
+		(net 26)
+	)
+	(segment
+		(start 132.74 66.84)
+		(end 132.71 66.81)
+		(width 0.2)
+		(layer "F.Cu")
+		(net 26)
+	)
+	(segment
+		(start 131.86 69.49)
+		(end 131.86 66.81)
+		(width 0.2)
+		(layer "F.Cu")
+		(net 30)
+	)
+	(segment
+		(start 130.74 70.61)
+		(end 131.86 69.49)
+		(width 0.2)
+		(layer "F.Cu")
+		(net 30)
+	)
+	(segment
 		(start 125.17 73.32)
 		(end 138.31 73.32)
 		(width 0.2)
 		(layer "F.Cu")
-		(net 44)
+		(net 42)
 	)
 	(segment
@@
 		(width 0.2)
 		(layer "F.Cu")
-		(net 45)
+		(net 43)
 	)
 	(segment
@@
 		(width 0.2)
 		(layer "F.Cu")
-		(net 45)
+		(net 43)
 	)
 	(segment
@@
 		(width 0.2)
 		(layer "F.Cu")
-		(net 45)
+		(net 43)
 	)
 	(via micro
@@
 		(drill 0.1)
 		(layers "F.Cu" "B.Cu")
-		(net 45)
+		(net 43)
 	)
 	(segment
@@
 		(width 0.2)
 		(layer "B.Cu")
-		(net 45)
+		(net 43)
 	)
 	(segment
@@
 		(width 0.2)
 		(layer "B.Cu")
-		(net 45)
+		(net 43)
 	)
 	(segment
@@
 		(width 0.2)
 		(layer "B.Cu")
-		(net 45)
+		(net 43)
 	)
 	(segment
@@
 		(width 0.2)
 		(layer "B.Cu")
-		(net 45)
+		(net 43)
 	)
 	(embedded_fonts no)
